Commit message: Add files via upload

File: grobot/urdf/grobot.urdf (robot description, URDF)
Before this commit: robot grobot, 7 links, 6 joints
Links:
- added link lidar, mass 0.01; collision cylinder length=0.05 radius=0.05; visual cylinder length=0.05 radius=0.05
Joints:
- added joint lidar_joint: type fixed, parent base_link, child lidar, origin xyz=0 0 0.1 rpy=0 0 0
